File: USB_Isolator.sch (EAGLE design)
At the start: 16 parts, among them J1 USB_A, J2 USB_MINI, U1 ADUM4160, U2 NUP4202, U3 NUP4202, U4 NMG0505SC

Commit message: 初めのテスト
Connections:
- net N$12 renamed DVDD
- net N$13 renamed DD_N
- net N$14 renamed DD_P
- net N$4 renamed UVDD
- net UD- renamed UD_N
- removed net UD+: J2.D+, R2.1, U2.IO6
- new net UD_P: J2.D+, R2.1, U2.IO3
Changed lines of the file:
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@@
 <class number="0" name="default" width="0" drill="0">
+</class>
+<class number="1" name="USB" width="0.381" drill="0.254">
+<clearance class="1" value="0.254"/>
+</class>
+<class number="2" name="Power" width="0.508" drill="0.508">
+<clearance class="2" value="0.762"/>
 </class>
 </classes>
@@
 </segment>
 </net>
-<net name="UVBUS" class="0">
+<net name="UVBUS" class="2">
 <segment>
 <pinref part="C3" gate="A" pin="2"/>
@@
 <pinref part="J2" gate="A" pin="VBUS"/>
 <wire x1="81.28" y1="127" x2="119.38" y2="127" width="0.1524" layer="91"/>
-<wire x1="119.38" y1="127" x2="121.92" y2="127" width="0.1524" layer="91"/>
-<wire x1="121.92" y1="127" x2="127" y2="127" width="0.1524" layer="91"/>
+<wire x1="119.38" y1="127" x2="127" y2="127" width="0.1524" layer="91"/>
 <wire x1="60.96" y1="93.98" x2="63.5" y2="93.98" width="0.1524" layer="91"/>
 <wire x1="63.5" y1="93.98" x2="63.5" y2="127" width="0.1524" layer="91"/>
@@
 <junction x="68.58" y="127"/>
 <junction x="81.28" y="127"/>
-<junction x="121.92" y="127"/>
 <junction x="119.38" y="104.14"/>
+<junction x="119.38" y="127"/>
 </segment>
 </net>
@@
 </segment>
 </net>
-<net name="N$4" class="0">
+<net name="UVDD" class="0">
 <segment>
 <pinref part="C4" gate="A" pin="2"/>
@@
 </segment>
 </net>
-<net name="UGND" class="0">
+<net name="UGND" class="2">
 <segment>
 <pinref part="U1" gate="A" pin="GND_1"/>
@@
 </segment>
 </net>
-<net name="UD-" class="0">
+<net name="UD_N" class="1">
 <segment>
 <pinref part="R1" gate="A" pin="1"/>
@@
 </segment>
 </net>
-<net name="UD+" class="0">
+<net name="UD_P" class="1">
 <segment>
 <pinref part="J2" gate="A" pin="D+"/>
 <pinref part="R2" gate="A" pin="1"/>
 <wire x1="60.96" y1="88.9" x2="76.2" y2="88.9" width="0.1524" layer="91"/>
-<pinref part="U2" gate="A" pin="IO6"/>
+<pinref part="U2" gate="A" pin="IO3"/>
 <wire x1="76.2" y1="88.9" x2="106.68" y2="88.9" width="0.1524" layer="91"/>
-<wire x1="76.2" y1="76.2" x2="76.2" y2="88.9" width="0.1524" layer="91"/>
+<wire x1="86.36" y1="60.96" x2="76.2" y2="88.9" width="0.1524" layer="91"/>
 <junction x="76.2" y="88.9"/>
 </segment>
@@
 </segment>
 </net>
-<net name="N$12" class="0">
+<net name="DVDD" class="0">
 <segment>
 <pinref part="C6" gate="A" pin="1"/>
@@
 </segment>
 </net>
-<net name="N$13" class="0">
+<net name="DD_N" class="1">
 <segment>
 <pinref part="R3" gate="A" pin="2"/>
@@
 </segment>
 </net>
-<net name="N$14" class="0">
+<net name="DD_P" class="1">
 <segment>
 <pinref part="R4" gate="A" pin="2"/>
@@
 </segment>
 </net>
-<net name="DGND" class="0">
+<net name="DGND" class="2">
 <segment>
 <pinref part="U1" gate="A" pin="GND2"/>
@@
 </segment>
 </net>
-<net name="DVBUS" class="0">
+<net name="DVBUS" class="2">
 <segment>
 <pinref part="U4" gate="A" pin="OUT+"/>
