File: USB_Isolator.brd (EAGLE design)
At the start: 60.2 x 25.1 mm, 16 parts, among them J1 USB_A, J2 USB_MINI, U1 ADUM4160, U2 NUP4202, U3 NUP4202, U4 NMG0505SC

Commit message: DRC調整
Routing:
- net UGND: vias 3 -> 4
Changed lines of the file:
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@@
 </class>
 </classes>
-<designrules name="default">
+<designrules name="default *">
 <description language="de">&lt;b&gt;EAGLE Design Rules&lt;/b&gt;
 &lt;p&gt;
@@
 <param name="mtCopper" value="0.035mm 0.035mm 0.035mm 0.035mm 0.035mm 0.035mm 0.035mm 0.035mm 0.035mm 0.035mm 0.035mm 0.035mm 0.035mm 0.035mm 0.035mm 0.035mm"/>
 <param name="mtIsolate" value="1.5mm 0.15mm 0.2mm 0.15mm 0.2mm 0.15mm 0.2mm 0.15mm 0.2mm 0.15mm 0.2mm 0.15mm 0.2mm 0.15mm 0.2mm"/>
-<param name="mdWireWire" value="8mil"/>
-<param name="mdWirePad" value="8mil"/>
-<param name="mdWireVia" value="8mil"/>
-<param name="mdPadPad" value="8mil"/>
-<param name="mdPadVia" value="8mil"/>
-<param name="mdViaVia" value="8mil"/>
+<param name="mdWireWire" value="6mil"/>
+<param name="mdWirePad" value="5mil"/>
+<param name="mdWireVia" value="5mil"/>
+<param name="mdPadPad" value="5mil"/>
+<param name="mdPadVia" value="5mil"/>
+<param name="mdViaVia" value="5mil"/>
 <param name="mdSmdPad" value="8mil"/>
 <param name="mdSmdVia" value="8mil"/>
@@
 <param name="mdViaViaSameLayer" value="8mil"/>
 <param name="mnLayersViaInSmd" value="2"/>
-<param name="mdCopperDimension" value="40mil"/>
+<param name="mdCopperDimension" value="10mil"/>
 <param name="mdDrill" value="8mil"/>
 <param name="mdSmdStop" value="0mil"/>
 <param name="msWidth" value="10mil"/>
-<param name="msDrill" value="24mil"/>
+<param name="msDrill" value="10mil"/>
 <param name="msMicroVia" value="9.99mm"/>
 <param name="msBlindViaRatio" value="0.5"/>
@@
 <param name="mvStopFrame" value="1"/>
 <param name="mvCreamFrame" value="0"/>
-<param name="mlMinStopFrame" value="4mil"/>
+<param name="mlMinStopFrame" value="6mil"/>
 <param name="mlMaxStopFrame" value="4mil"/>
 <param name="mlMinCreamFrame" value="0mil"/>
@@
 <via x="10.16" y="18.542" extent="1-16" drill="0.6"/>
 <via x="18.796" y="9.398" extent="1-16" drill="0.6"/>
-<wire x1="14.351" y1="11.491" x2="18.796" y2="9.398" width="0" layer="19" extent="1-1"/>
-<wire x1="2.08" y1="9.393" x2="7.58" y2="9.393" width="0" layer="19" extent="1-1"/>
+<via x="10.16" y="10.922" extent="1-16" drill="0.6"/>
 </signal>
 <signal name="UD_N" class="1">
@@
 <via x="37.846" y="10.668" extent="1-16" drill="0.6"/>
 <via x="42.672" y="20.32" extent="1-16" drill="0.6"/>
-<wire x1="37.211" y1="19.954" x2="42.672" y2="20.32" width="0" layer="19" extent="1-1"/>
-<wire x1="35.306" y1="19.924" x2="37.196" y2="19.939" width="0" layer="19" extent="1-1"/>
+<wire x1="37.196" y1="19.939" x2="35.306" y2="19.924" width="0" layer="19" extent="1-1"/>
 </signal>
 <signal name="DVBUS" class="2">
@@
 <via x="14.351" y="8.509" extent="1-16" drill="0.254"/>
 </signal>
-<signal name="N$5">
-<via x="10.16" y="10.922" extent="1-16" drill="0.6"/>
-</signal>
 </signals>
+<errors>
+</errors>
 </board>
 </drawing>
